Commit message: fix(tasks): remove computer vision tasks, add lidar/kinematic alternatives and add 2D lidar to basic_mobile_robot
- Replace vision/camera tasks with lidar target tracking and Kanayama Lyapunov controller (Module 1)
- Replace YouBot vision task with 8-DOF redundancy resolution in null-space (Module 2)
- Refine Mecanum task to forward/inverse 4-wheel kinematics and odometry reconstruction
- Add 2D lidar sensor (libgazebo_ros_ray_sensor.so) to basic_mobile_bot.xacro.urdf
- Add explicit note on kinematic grasping for Pick & Place in ODE

File: src/basic_mobile_robot/models/basic_mobile_bot.xacro.urdf (robot description, URDF)
Before this commit: robot basic_mobile_bot, 5 links, 4 joints
Links:
- added link lidar_link; collision cylinder length=0.05 radius=0.05; visual cylinder length=0.05 radius=0.05
Joints:
- added joint lidar_joint: type fixed, parent base_link, child lidar_link, origin xyz=0.215 0 0.125 rpy=0 0 0
